File: YWS_clock/YWS_clock.kicad_sch (KiCad schematic)
At the start: 32 parts, among them U2 ATmega328-PU, Y1 Crystal_16MHz

Commit message: Update Buzzer and joystick
Connections:
- net VCC: no longer R?.2, R?.2, R?.2, R?.2, U?.18 (ISET), U?.18 (ISET), U?.18 (ISET), U?.18 (ISET)
- new net: R?.2, U?.18 (ISET) (x4)
Other:
- moved on the sheet: R?

Commit message: Update button
Parts:
- added BT1: Battery_Cell, footprints:BatteryHolder_Keystone_106_1x20mm, symbol HPS:Battery_Cell
- added BZ1: Buzzer, footprints:Buzzer_TDK_PS1240P02BT_D12.2mm_H6.5mm, symbol HPS:Buzzer
- added C5: C_0805_0.1uf, footprints:C_0805_2012Metric, symbol HPS:C_0805_0.1uf
- added C6, C7: C_0805_1uf, footprints:C_0805_2012Metric, symbol HPS:C_0805_1uf
- added D1: LED_0805, footprints:LED_0805_2012Metric, symbol HPS:LED_0805
- added J1, J3: Conn_01x06, footprints:PinHeader_1x06_P2.54mm_Vertical, symbol HPS:Conn_01x06
- added J2: PJ-102AH, footprints:PJ-102AH, symbol HPS:PJ-102AH
- added R11, R12, R13, R14: R_0805_10K, footprints:R_0805_2012Metric, symbol HPS:R_0805_10K
- added R15: PhotoconductivePhotocell, footprints:R_LDR_4.9x4.2mm_P2.54mm_Vertical, symbol HPS:PhotoconductivePhotocell
- added R2, R5, R6: R_0805_2.2K, footprints:R_0805_2012Metric, symbol HPS:R_0805_2.2K
- added R3, R4: R_0805_47, footprints:R_0805_2012Metric, symbol HPS:R_0805_47
- added SW1, SW2, SW3, SW4: Omron_B3F_SPST, footprints:SW_SPST_Omron_B3FS-100xP, symbol HPS:Omron_B3F_SPST
- added U1: L7805, footprints:TO-220-3_Horizontal_TabDown, symbol HPS:L7805
- added Y2: Crystal_16MHz, footprints:Crystal_SMD_HC49-SD, symbol HPS:Crystal_16MHz
- gave numbers to parts that had none: 21
Connections:
- net GND: now also U3.4 (GND), BT1.2 (-), C6.2, C7.2, D1.1 (K), J1.1 (Pin_1), J1.2 (Pin_2), J2.2 (OUT), J3.3 (Pin_3), R11.2, R12.2, R13.2, SW1.1 (A), SW1.2 (A), U1.2 (GND)
- net LED_SCK: now also U2.15 (PB1), U2.18 (PB4), R2.1; no longer U2.17 (PB3), U2.19 (PB5)
- net RESET: now also C5.1, SW1.3 (B), SW1.4 (B)
- net RXD: now also U2.12 (PD6), R3.2; no longer U2.2 (PD0)
- net TXD: now also U2.13 (PD7), R4.1; no longer U2.4 (PD2)
- net VCC: now also U3.8 (VCC), BZ1.1 (-), C7.1, J3.2 (Pin_2), R5.1, R6.1, SW2.1 (A), SW2.2 (A), SW3.1 (A), SW3.2 (A), SW4.1 (A), SW4.2 (A), U1.3 (OUT)
- net at U5.12 (LOAD): now also U2.16 (PB2), U4.12 (LOAD), U6.12 (LOAD), U7.12 (LOAD)
- net at U5.13 (CLK): now also U2.19 (PB5), U4.13 (CLK), U6.13 (CLK), U7.13 (CLK)
- net at U3.1 (X1): now also Y2.1
- net at U3.2 (X2): now also Y2.2
- net at U3.3 (VBAT): now also BT1.1 (+)
- net at U3.5 (SDA): now also U2.3 (PD1), R5.2
- net at U3.6 (SCL): now also U2.2 (PD0), R6.2
- net at U4.1 (DIN): now also U2.17 (PB3)
- net at U2.11 (PD5): now also J3.6 (Pin_6)
- net at U2.23 (PC0): now also J3.4 (Pin_4)
- net at U2.24 (PC1): now also J3.5 (Pin_5)
- net at U2.25 (PC2): now also SW2.3 (B)
- net at U2.26 (PC3): now also SW3.3 (B)
- net at U2.27 (PC4): now also SW4.3 (B)
- net at U2.5 (PD3): now also BZ1.2 (+)
- net at U2.6 (PD4): now also R14.2
- new net: C6.1, J2.1 (POLE), U1.1 (IN)
- new net: R15.1, U2.4 (PD2)
- new net: R14.1, R15.2
- new net: C5.2, J1.6 (Pin_6)
- new net: J1.5 (Pin_5), R3.1
- new net: J1.4 (Pin_4), R4.2
- new net: R13.1, SW4.4 (B)
- new net: D1.2 (A), R2.2
- new net: R11.1, SW2.4 (B)
- new net: R12.1, SW3.4 (B)
- no-connect marks 0 -> 6
Other:
- note added: "DS1307"
- note added: "LED"
- note added: "Power Input"
- note added: "Serial"
- note added: "Vf = 2v Vr = 3v 10mcd @ 1.35mA therefore R = 2.2K0hm"
- moved on the sheet: C1, C10, C11, C12, C13, C14, C15, C2, C3, C4, C8, C9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

Commit message: Update with PCB layout
Parts:
- added D6: LED_0805, footprints:LED_0805_2012Metric, symbol HPS:LED_0805
- added R16: R_0805_2.2K, footprints:R_0805_2012Metric, symbol HPS:R_0805_2.2K
Connections:
- net GND: now also D6.1 (K)
- net LED_SCK: now also R16.1
- new net: D6.2 (A), R16.2
- no-connect marks 6 -> 7
Other:
- note added: "Yuwei Sun's clock with dot matrix"
- moved on the sheet: C2
